File: hardware/cm4_adc.brd (EAGLE design)
At the start: 82.1 x 78.8 mm, 16 parts, among them J2 PJ-102A, Q1 2N7002, Q2 2.5A/30V/105mΩ, U1 ADT7420UCPZ-RL7

Commit message: Major file changes
Changes to Schematic, Part number updates etc.
Parts:
- Q1: value 2N7002 -> XP151A12A2MR-G
Changed lines of the file:
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@@
 <attribute name="VALUE" x="55.245" y="64.897" size="0.6096" layer="27" font="vector" ratio="20" align="top-center"/>
 </element>
-<element name="Q1" library="SparkFun-DiscreteSemi" library_urn="urn:adsk.eagle:library:514" package="SOT323" package3d_urn="urn:adsk.eagle:package:38456/1" value="2N7002" x="70.104" y="68.961" smashed="yes">
+<element name="Q1" library="SparkFun-DiscreteSemi" library_urn="urn:adsk.eagle:library:514" package="SOT323" package3d_urn="urn:adsk.eagle:package:38456/1" value="XP151A12A2MR-G" x="70.104" y="68.961" smashed="yes">
 <attribute name="NAME" x="67.691" y="69.469" size="1.016" layer="25" font="vector" ratio="20" rot="R180" align="bottom-center"/>
 <attribute name="PROD_ID" value="TRANS-11151" x="70.104" y="68.961" size="1.778" layer="27" display="off"/>
@@
 <vertex x="9.0805" y="22.9235"/>
 <vertex x="9.906" y="23.876"/>
-<vertex x="9.906" y="23.876"/>
 </polygon>
